Commit message: updated nodes

File: objects/box_1.urdf (robot description, URDF)
Before this commit: robot simple_box, 1 links, 0 joints
Links:
- link my_box: geometry collision box size=0.3 0.3 0.11; visual box size=0.3 0.3 0.11

Commit message: unclean results

File: objects/box_1.urdf (robot description, URDF)
Before this commit: robot simple_box, 1 links, 0 joints
Links:
- link my_box: mass 1.0 -> 3.0; geometry collision box size=0.3 0.3 0.011; visual box size=0.3 0.3 0.05
